File: lora_pager.kicad_pcb (KiCad board)
At the start: 2 copper layers, 97.2 x 66 mm, 28 parts, among them J1 USB_C_Receptacle_USB2.0_14P, Q2 AO3400A, SW3 TS-1089S-02526, SW4 TS-1089S-02526, U1 E22-900M30S, U2 HS17QS178RX, U3 ESP32-S3-MINI-1, U4 AMS1117-3.3

Commit message: sus commit
Parts:
- removed ?: , clipboard:e001904d-a08e-4160-8a50-c56007e02e2b
- removed C12, C9: 10uF, Capacitor_SMD:C_1206_3216Metric_Pad1.33x1.80mm_HandSolder
- removed D10: 1N4148WS, Diode_SMD:D_SOD-323_HandSoldering
- removed FPC1: 5034801000, easyeda2kicad:FPC-SMD_5034801000
- removed LS1: Buzzer, easyeda2kicad:BUZ-SMD_4P-L8.5-W8.5-P8.50-BR
- removed Q2: AO3400A, Package_TO_SOT_SMD:SOT-23_Handsoldering
- removed R15: 10k, Resistor_SMD:R_0805_2012Metric_Pad1.20x1.40mm_HandSolder
- removed R16: 10, Resistor_SMD:R_0603_1608Metric_Pad0.98x0.95mm_HandSolder
- removed U2: HS17QS178RX, easyeda2kicad:OLED-SMD_10P-P0.50_HS17QS178RX
- removed U4: AMS1117-3.3, Package_TO_SOT_SMD:SOT-223-3_TabPin2
- added BT3: li-ion, Connector_JST:JST_PH_B2B-PH-K_1x02_P2.00mm_Vertical, F.Cu at (157.8, 112.5)
- added C10: 10pF, Capacitor_SMD:C_0402_1005Metric_Pad0.74x0.62mm_HandSolder, F.Cu at (163.4, 137.8)
- added C11: 22uF, Capacitor_SMD:C_0805_2012Metric_Pad1.18x1.45mm_HandSolder, F.Cu at (147.2, 141.4)
- added C13: 22uF, Capacitor_SMD:C_0805_2012Metric_Pad1.18x1.45mm_HandSolder, F.Cu at (147.2, 144.5)
- added C14: 22uF, Capacitor_SMD:C_0805_2012Metric_Pad1.18x1.45mm_HandSolder, F.Cu at (147.2, 147.5)
- added C3: 10uF, Capacitor_SMD:C_0805_2012Metric_Pad1.18x1.45mm_HandSolder, F.Cu at (147.2, 132.4)
- added C4: 10uF, Capacitor_SMD:C_0805_2012Metric_Pad1.18x1.45mm_HandSolder, F.Cu at (147.2, 135.4)
- added C5: 1uF, Capacitor_SMD:C_0402_1005Metric_Pad0.74x0.62mm_HandSolder, F.Cu at (163.4, 131.9)
- added C6: 1uF, Capacitor_SMD:C_0402_1005Metric_Pad0.74x0.62mm_HandSolder, F.Cu at (163.4, 133.9)
- added C7: 10nF, Capacitor_SMD:C_0402_1005Metric_Pad0.74x0.62mm_HandSolder, F.Cu at (163.4, 135.8)
- added C8: 10uF, Capacitor_SMD:C_0805_2012Metric_Pad1.18x1.45mm_HandSolder, F.Cu at (147.2, 138.4)
- added D3: Red, LED_SMD:LED_0805_2012Metric_Pad1.15x1.40mm_HandSolder, F.Cu at (156.4, 140.6)
- added D4: Green, LED_SMD:LED_0805_2012Metric_Pad1.15x1.40mm_HandSolder, F.Cu at (156.4, 143.7)
- added F2: 4A/8A, Fuse:Fuse_1812_4532Metric_Pad1.30x3.40mm_HandSolder, F.Cu at (152.5, 107.0)
- added L1: 1uH, Inductor_SMD_Wurth:L_Wurth_WE-LQSH-4020, F.Cu at (127.2, 103.2)
- added LS2: Speaker, easyeda2kicad:BUZ-SMD_4P-L13.0-W13.0-P11.4-BL, F.Cu at (152.8, 59.2)
- added Q1: AOD403, Package_TO_SOT_SMD:TO-252-2, F.Cu at (185.1, 124.2)
- added Q3: AO3400A, Package_TO_SOT_SMD:SOT-23_Handsoldering, F.Cu at (145.5, 125.8)
- added Q4: AOD403, Package_TO_SOT_SMD:TO-252-2, F.Cu at (194.2, 124.4)
- added R10: 2.2k, Resistor_SMD:R_0603_1608Metric_Pad0.98x0.95mm_HandSolder, F.Cu at (151.8, 140.4)
- added R11: 316k, Resistor_SMD:R_0402_1005Metric_Pad0.72x0.64mm_HandSolder, F.Cu at (160.4, 144.1)
- added R12: 100k, Resistor_SMD:R_0603_1608Metric_Pad0.98x0.95mm_HandSolder, F.Cu at (151.8, 142.9)
- added R13: 1M, Resistor_SMD:R_0402_1005Metric_Pad0.72x0.64mm_HandSolder, F.Cu at (153.6, 72.1)
- added R14: 1k, Resistor_SMD:R_0402_1005Metric_Pad0.72x0.64mm_HandSolder, F.Cu at (150.4, 124.3)
- added R18: 10k, Resistor_SMD:R_0402_1005Metric_Pad0.72x0.64mm_HandSolder, F.Cu at (150.4, 126.3)
- added R19: 470k, Resistor_SMD:R_0603_1608Metric_Pad0.98x0.95mm_HandSolder, F.Cu at (151.8, 145.4)
- added R5: 1k, Resistor_SMD:R_0402_1005Metric_Pad0.72x0.64mm_HandSolder, F.Cu at (160.4, 140.1)
- added R8: 1k, Resistor_SMD:R_0402_1005Metric_Pad0.72x0.64mm_HandSolder, F.Cu at (160.4, 142.1)
- added SW2: SS-12D10L5, easyeda2kicad:SW-TH_SS-12D10L5, F.Cu at (158.8, 102.3)
- added SW5: TS-1089S-02526, easyeda2kicad:SW-SMD_4P-L4.2-W3.3-P2.15-LS5.1, F.Cu at (120.1, 84.7)
- added SW6: TS-1089S-02526, easyeda2kicad:SW-SMD_4P-L4.2-W3.3-P2.15-LS5.1, F.Cu at (111.4, 84.7)
- added SW7: TS-1089S-02526, easyeda2kicad:SW-SMD_4P-L4.2-W3.3-P2.15-LS5.1, F.Cu at (128.8, 84.7)
- added SW8: TS-1089S-02526, easyeda2kicad:SW-SMD_4P-L4.2-W3.3-P2.15-LS5.1, F.Cu at (137.4, 84.7)
- added SW9: TS-1089S-02526, easyeda2kicad:SW-SMD_4P-L4.2-W3.3-P2.15-LS5.1, F.Cu at (146.1, 84.7)
- added U10: ME6211C33M5, Package_TO_SOT_SMD:SOT-23-5, F.Cu at (130.5, 110.8)
- added U11: TPS61230ARNSR, easyeda2kicad:VQFN-7_L2.1-W2.1-P0.50-BL, F.Cu at (131.2, 103.5)
- added U13: LTC4412xS6, Package_TO_SOT_SMD:TSOT-23-6, F.Cu at (147.2, 96.0)
- added U14: MAX98357A, Package_DFN_QFN:TQFN-16-1EP_3x3mm_P0.5mm_EP1.23x1.23mm, F.Cu at (152.8, 68.7)
- added U5: HS96L03W2C03, easyeda2kicad:OLED-TH_L27.8-W27.2-P2.54_C9900033791, F.Cu at (128.5, 55.0)
- added U9: TP4056-42-ESOP8, Package_SO:SOIC-8-1EP_3.9x4.9mm_P1.27mm_EP2.41x3.3mm_ThermalVias, F.Cu at (143.8, 109.1)
- F1: value 500ma/1A -> 1A/1.8A
- moved SW3 104.3 mm to (67.8, 56.0), turned to 90 degrees
- moved SW4 87.1 mm to (67.8, 83.2), turned to 90 degrees
- moved F1 80.0 mm to (92.0, 61.8), turned to -90 degrees
- moved R9 21.7 mm to (111.0, 126.2)
- moved J1 4.18 mm to (88.8, 54.0)
Connections:
- D21 pad 2: +5V -> VBUS
- F1 pad 2: +5V -> VBUS
- U3 pad 18: unconnected-(U3-IO14-Pad18) -> Net-(U3-IO14)
- U3 pad 19: unconnected-(U3-IO15-Pad19) -> Net-(U3-IO15)
- U3 pad 20: unconnected-(U3-IO16-Pad20) -> Net-(U3-IO16)
- U3 pad 21: unconnected-(U3-IO17-Pad21) -> Net-(U3-IO17)
- U3 pad 22: unconnected-(U3-IO18-Pad22) -> Net-(U3-IO18)
- U3 pad 25: unconnected-(U3-IO21-Pad25) -> SDA
- U3 pad 26: unconnected-(U3-IO26-Pad26) -> SCL
- U3 pad 28: unconnected-(U3-IO33-Pad28) -> EN
- U3 pad 29: unconnected-(U3-IO34-Pad29) -> BACKLIGHT
- U3 pad 31: unconnected-(U3-IO35-Pad31) -> BUZZER
- U3 pad 32: unconnected-(U3-IO36-Pad32) -> DIN
- U3 pad 33: unconnected-(U3-IO37-Pad33) -> BCLK
- U3 pad 34: BUZZER -> LRCLK

Commit message: Finished first rough draft
Parts:
- removed Q3: AO3400A, Package_TO_SOT_SMD:SOT-23_Handsoldering
- removed R14: 1k, Resistor_SMD:R_0402_1005Metric_Pad0.72x0.64mm_HandSolder
- removed R18: 10k, Resistor_SMD:R_0402_1005Metric_Pad0.72x0.64mm_HandSolder
- moved Q4 107.2 mm to (108.8, 59.5), turned to -90 degrees
- moved C6 98.7 mm to (80.1, 80.9), turned to 180 degrees
- moved C5 94.3 mm to (80.4, 87.2), turned to -90 degrees
- moved R17 89.1 mm to (85.6, 60.5)
- moved C18 86.2 mm to (86.2, 58.4), turned to 90 degrees
- moved D15 76.0 mm to (96.5, 62.2), turned to -90 degrees
- moved D20 74.8 mm to (98.8, 64.4), turned to 90 degrees
- moved C14 74.7 mm to (124.7, 76.2)
- moved R7 74.6 mm to (95.3, 60.4), turned to 180 degrees
- moved D21 74.3 mm to (104.2, 64.6)
- moved D1 73.3 mm to (83.4, 80.0), turned to 180 degrees
- moved R6 70.0 mm to (99.4, 61.7), turned to -90 degrees
- moved C16 62.2 mm to (80.8, 89.0), turned to 180 degrees
- moved U10 56.9 mm to (80.4, 83.9), turned to 90 degrees
- moved R19 56.2 mm to (161.0, 89.9), turned to 90 degrees
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Connections:
- Q4 pad 1: GND -> Net-(Q4-G)
- R13 pad 1: +3V3 -> +5V
- R19 pad 2: GND -> Net-(Q4-G)
- U1 pad 13: DIO1 -> unconnected-(U1-DIO1-Pad13)
- U1 pad 8: DIO2 -> unconnected-(U1-DIO2-Pad8)
- U13 pad 4: GND -> Net-(Q4-G)
Routing:
- net Vin: track 0.00 -> 180.8 mm, vias 0 -> 2
- net +5V: track 0.00 -> 102.7 mm, vias 0 -> 4
- net VBUS: track 0.00 -> 91.1 mm
- net Net-(Q4-G): track 0.00 -> 86.0 mm
- net +3V3: track 0.00 -> 82.0 mm, vias 0 -> 2
- net EN: track 0.00 -> 71.3 mm, vias 0 -> 4
- net LRCLK: track 0.00 -> 67.3 mm, vias 0 -> 2
- net BCLK: track 0.00 -> 66.1 mm, vias 0 -> 2
- net DIN: track 0.00 -> 65.5 mm, vias 0 -> 2
- net Net-(U3-IO18): track 0.00 -> 60.6 mm, vias 0 -> 2
- net Net-(U3-IO17): track 0.00 -> 51.8 mm, vias 0 -> 2
- net GND: track 0.00 -> 50.5 mm, vias 0 -> 17
- net SDA: track 0.00 -> 49.3 mm, vias 0 -> 2
- net SCL: track 0.00 -> 47.0 mm, vias 0 -> 2
- net TXEN: track 0.00 -> 43.4 mm, vias 0 -> 2
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- added copper zone on F.Cu, net GND
- added copper zone on F.Cu, net Vin
Other:
- board size 97.2 x 66 mm -> 85 x 66 mm
- board text added: "A"
- board text added: "B"
- board text added: "BOOT"
- board text added: "C"
- board text added: "D"
- board text added: "E"
- board text added: "LoRa Pager"
- board text added: "RESET"

Commit message: almost done :siren-thumbsup:
Parts:
- removed the R17 at (85.6, 60.5)
- added BT2: li-ion, easyeda2kicad:BATTERY-SMD_18650-1S-L77.1-W20.7-1, B.Cu at (117.3, 82.9)
- added D3: D_TVS, Diode_SMD:D_SOD-923, F.Cu at (148.3, 108.0)
- added D4: D_TVS, Diode_SMD:D_SOD-923, F.Cu at (149.1, 80.2)
- added D5: D_TVS, Diode_SMD:D_SOD-923, F.Cu at (135.8, 64.5)
- added D6: D_TVS, Diode_SMD:D_SOD-923, F.Cu at (128.8, 108.5)
- added D7: D_TVS, Diode_SMD:D_SOD-923, F.Cu at (95.8, 66.8)
- added R10: 10k, Resistor_SMD:R_0402_1005Metric_Pad0.72x0.64mm_HandSolder, F.Cu at (120.1, 81.0)
- added R11: 10k, Resistor_SMD:R_0402_1005Metric_Pad0.72x0.64mm_HandSolder, F.Cu at (133.0, 81.2)
- added R12: 10k, Resistor_SMD:R_0402_1005Metric_Pad0.72x0.64mm_HandSolder, F.Cu at (141.8, 83.2)
- added R13: 10k, Resistor_SMD:R_0402_1005Metric_Pad0.72x0.64mm_HandSolder, F.Cu at (146.0, 81.0)
- added R14: 10k, Resistor_SMD:R_0402_1005Metric_Pad0.72x0.64mm_HandSolder, F.Cu at (87.1, 60.2)
- added R2: 10k, Resistor_SMD:R_0402_1005Metric_Pad0.72x0.64mm_HandSolder, F.Cu at (128.4, 56.5)
- added R4: 10k, Resistor_SMD:R_0402_1005Metric_Pad0.72x0.64mm_HandSolder, F.Cu at (128.2, 57.8)
- added R9: 10k, Resistor_SMD:R_0402_1005Metric_Pad0.72x0.64mm_HandSolder, F.Cu at (116.5, 83.7)
- added U6: INA3221, Package_DFN_QFN:Texas_RGV0016A_VQFN-16-1EP_4x4mm_P0.65mm_EP2.1x2.1mm, F.Cu at (155.3, 86.0)
- renumbered BT3 to BT1, C8 to C1, C13 to C10, C17 to C11, C18 to C12, C16 to C13, C7 to C2, C5 to C3, C10 to C4, C4 to C5, C11 to C6, C14 to C7, C3 to C8, C6 to C9, D4 to D1, D20 to D10, D21 to D11, D3 to D2, D1 to D8, D15 to D9, F2 to F1, F1 to F2, LS2 to LS1, Q4 to Q1, Q1 to Q2, R8 to R1, R13 to R15, R9 to R16, R6 to R17, R7 to R18, R5 to R3, R11 to R5, R12 to R6, R10 to R7, R19 to R8, SW2 to SW1, SW5 to SW2, SW6 to SW3, SW7 to SW4, SW8 to SW5, SW9 to SW6, SW3 to SW7, SW4 to SW8, U11 to U1, U13 to U2, U9 to U3, U5 to U4, U10 to U5, U1 to U7, U3 to U8, U14 to U9
Connections:
- R8 pad 1: Net-(U13-SENSE) -> Vin
- U2 pad 6: Net-(U13-SENSE) -> Vin
- U8 pad 11: DIO2 -> unconnected-(U8-IO7-Pad11)
- U8 pad 29: BACKLIGHT -> unconnected-(U8-IO34-Pad29)
- U8 pad 31: BUZZER -> unconnected-(U8-IO35-Pad31)
- U8 pad 8: DIO1 -> unconnected-(U8-IO4-Pad8)
Routing:
- net +3V3: track 82.0 -> 185.1 mm, vias 2 -> 6
- net SDA: track 49.3 -> 96.2 mm, vias 2 -> 4
- net SCL: track 47.0 -> 87.9 mm, vias 2 -> 3
- net +BATT: track 29.1 -> 48.5 mm, vias 0 -> 1
- net Vin: track 180.8 -> 199.1 mm
- net GND: track 50.5 -> 55.4 mm, vias 17 -> 65
- net Net-(BT1-+): track 9.78 -> 12.5 mm, vias 0 -> 1
- net Net-(U8-IO18): track 60.6 -> 63.1 mm
- net Net-(U8-IO14): track 25.8 -> 28.1 mm
- net Net-(U13-SENSE): track 2.27 -> 0.00 mm
- net Net-(U8-IO15): track 34.1 -> 36.3 mm
- net Net-(U8-IO16): track 43.2 -> 45.0 mm
- net Net-(U8-IO17): track 51.8 -> 53.6 mm
- net +5V: track 102.7 -> 103.9 mm
- added copper zone on B.Cu, net GND
Other:
- board text added: "DO NOT CONNECT TWO BATTERIES AT THE SAME TIME"
- board text added: "v1.0 2025-03-15"

Commit message: Final product: version 1 has been ordered
Parts:
- added J3: Conn_01x05_Socket, Connector_PinHeader_2.54mm:PinHeader_1x05_P2.54mm_Vertical, F.Cu at (80.0, 53.0)
- L1: footprint Inductor_SMD_Wurth:L_Wurth_WE-LQSH-4020 -> 74438356010:WE-MAPI_4020
- moved D7 2.62 mm to (96.7, 64.3), turned to 90 degrees
- moved SW7 2.45 mm to (81.5, 60.8)
- moved R14 1.31 mm to (86.2, 61.2)
- moved C12 1.25 mm to (85.5, 59.4)
- moved R11 0.50 mm to (133.0, 81.8)
Connections:
- U3 pad 1: unconnected-(U3-TEMP-Pad1) -> GND
- U8 pad 25: SDA -> unconnected-(U8-IO21-Pad25)
- U8 pad 26: SCL -> unconnected-(U8-IO26-Pad26)
- U8 pad 27: unconnected-(U8-IO47-Pad27) -> IO47
- U8 pad 29: unconnected-(U8-IO34-Pad29) -> SDA
- U8 pad 30: unconnected-(U8-IO48-Pad30) -> IO48
- U8 pad 31: unconnected-(U8-IO35-Pad31) -> SCL
- U8 pad 36: unconnected-(U8-IO40-Pad36) -> IO40
- U8 pad 37: unconnected-(U8-IO41-Pad37) -> IO41
- U8 pad 38: unconnected-(U8-IO42-Pad38) -> IO42
Routing:
- net IO42: track 0.00 -> 19.6 mm, vias 0 -> 1
- net IO47: track 0.00 -> 18.7 mm, vias 0 -> 1
- net IO41: track 0.00 -> 16.2 mm, vias 0 -> 2
- net IO48: track 0.00 -> 15.4 mm, vias 0 -> 1
- net IO40: track 0.00 -> 11.9 mm, vias 0 -> 2
- net GND: track 55.4 -> 47.2 mm, vias 65 -> 73
- net SCL: track 87.9 -> 93.3 mm
- net Net-(BT1-+): track 12.5 -> 15.5 mm, vias 1 -> 3
- net Net-(U8-EN): track 12.1 -> 9.89 mm
- net SDA: track 96.2 -> 97.4 mm
- net +5V: track 103.9 -> 105.0 mm
- net +3V3: track 185.1 -> 184.2 mm
- net Net-(U8-IO16): track 45.0 -> 44.5 mm
Other:
- board text added: "42-41-40-47-48"
- board text added: "Designed by Alex Park: parkalex.dev https://github.com/alx-alexpark/lora-pager"
- board text added: "v1.0 2025-03-14"
- board text removed: "v1.0 2025-03-15"
