File: lora_pager.kicad_sch (KiCad schematic)
At the start: 61 parts, among them J1 USB_C_Receptacle_USB2.0_14P, Q1 AOD403, Q2 AO3400A, SW3 TS-1089S-02526, SW4 TS-1089S-02526, U1 E22-900M30S, U10 ME6211C33M5, U11 TPS61230ARNSR, U12 XB8089D0, U2 HS17QS178RX, U3 ESP32-S3-MINI-1, U5 HS20HS072RX, U6 BQ76905RGRR, U7 SIRA60DP-T1-GE3, U8 SIRA60DP-T1-GE3, U9 TP4056-42-ESOP8

Commit message: sus commit
Parts:
- removed D2: SS14, symbol Device:D_Schottky
- removed U5: HS20HS072RX, easyeda2kicad:OLED-SMD_HS20HS072RX, symbol easyeda2kicad:HS20HS072RX
- added C14: 22uF, Capacitor_SMD:C_0805_2012Metric_Pad1.18x1.45mm_HandSolder, symbol Device:C_Small
- added F2: 4A/8A, Fuse:Fuse_1812_4532Metric_Pad1.30x3.40mm_HandSolder, symbol Device:Polyfuse_Small
- added LS2: Speaker, easyeda2kicad:BUZ-SMD_4P-L13.0-W13.0-P11.4-BL, symbol Device:Speaker
- added Q3: AO3400A, Package_TO_SOT_SMD:SOT-23_Handsoldering, symbol Device:Q_NMOS_GSD
- added Q4: AOD403, Package_TO_SOT_SMD:TO-252-2, symbol Transistor_FET:Q_PMOS_GDS
- added R14: 1k, Resistor_SMD:R_0402_1005Metric_Pad0.72x0.64mm_HandSolder, symbol Device:R
- added R18: 10k, Resistor_SMD:R_0402_1005Metric_Pad0.72x0.64mm_HandSolder, symbol Device:R
- added R19: 470k, Resistor_SMD:R_0603_1608Metric_Pad0.98x0.95mm_HandSolder, symbol Device:R_Small
- added SW2: SS-12D10L5, easyeda2kicad:SW-TH_SS-12D10L5, symbol Switch:SW_SPDT
- added SW5, SW6, SW7, SW8, SW9: TS-1089S-02526, easyeda2kicad:SW-SMD_4P-L4.2-W3.3-P2.15-LS5.1, symbol Switch:SW_Push
- added U13: LTC4412xS6, Package_TO_SOT_SMD:TSOT-23-6, symbol Power_Management:LTC4412xS6
- added U14: MAX98357A, Package_DFN_QFN:TQFN-16-1EP_3x3mm_P0.5mm_EP1.23x1.23mm, symbol Audio:MAX98357A
- added U15: KLJ-01304T-08R07W, easyeda2kicad:BUZ-SMD_4P-L13.0-W13.0-P11.4-BL, symbol easyeda2kicad:KLJ-01304T-08R07W
- added U4: HS17QS178RX, easyeda2kicad:FPC-SMD_5034801000, symbol easyeda2kicad:HS17QS178RX
- added U5: HS96L03W2C03, easyeda2kicad:OLED-TH_L27.8-W27.2-P2.54_C9900033791, symbol easyeda2kicad:HS96L03W2C03
- BT1, BT2, C1, C2, R1, R2, R3, R4, U12, U6, U7, U8: now not fitted
- BT3: footprint (none) -> Connector_JST:JST_PH_B2B-PH-K_1x02_P2.00mm_Vertical; LCSC Part (none) -> C131337
- C10: footprint (none) -> Capacitor_SMD:C_0402_1005Metric_Pad0.74x0.62mm_HandSolder; LCSC Part (none) -> C106199
- C11, C13: footprint (none) -> Capacitor_SMD:C_0805_2012Metric_Pad1.18x1.45mm_HandSolder; LCSC Part (none) -> C5674
- C3, C4, C8: footprint (none) -> Capacitor_SMD:C_0805_2012Metric_Pad1.18x1.45mm_HandSolder; LCSC Part (none) -> C15850
- C5, C6: footprint (none) -> Capacitor_SMD:C_0402_1005Metric_Pad0.74x0.62mm_HandSolder; LCSC Part (none) -> C14445
- C7: footprint (none) -> Capacitor_SMD:C_0402_1005Metric_Pad0.74x0.62mm_HandSolder; LCSC Part (none) -> C60133
- D10, FPC1, LS1, Q2, R15, R16, U2: now not fitted; now left out of the parts list
- D3: footprint (none) -> LED_SMD:LED_0805_2012Metric_Pad1.15x1.40mm_HandSolder; LCSC Part (none) -> C84256
- D4: footprint (none) -> LED_SMD:LED_0805_2012Metric_Pad1.15x1.40mm_HandSolder; LCSC Part (none) -> C2297
- F1: value 500ma/1A -> 1A/1.8A; LCSC Part C720075 -> C70082
- L1: footprint (none) -> Inductor_SMD_Wurth:L_Wurth_WE-LQSH-4020; Digikey (none) -> 732-8228-2-ND; LCSC Part (none) -> X
- Q1: footprint (none) -> Package_TO_SOT_SMD:TO-252-2
- R10: footprint (none) -> Resistor_SMD:R_0603_1608Metric_Pad0.98x0.95mm_HandSolder; LCSC Part (none) -> C114662
- R11: value 386k -> 316k; footprint (none) -> Resistor_SMD:R_0402_1005Metric_Pad0.72x0.64mm_HandSolder; LCSC Part (none) -> C2998151
- R12: footprint (none) -> Resistor_SMD:R_0603_1608Metric_Pad0.98x0.95mm_HandSolder; LCSC Part (none) -> C14675
- R13: value 10k -> 1M; footprint (none) -> Resistor_SMD:R_0402_1005Metric_Pad0.72x0.64mm_HandSolder; LCSC Part (none) -> C138033
- R5, R8: footprint (none) -> Resistor_SMD:R_0402_1005Metric_Pad0.72x0.64mm_HandSolder; LCSC Part (none) -> C106235
- U10: LCSC Part (none) -> C82942
- U3: LCSC Part (none) -> C2913206
- U9: LCSC Part (none) -> C16581
Connections:
- net +3V3: now also R13.1, U4.8 (VDD3.3V), U4.9 (LEDA), U5.2 (VCC)
- net +5V: now also U14.7 (VDD), U14.8 (VDD)
- net +BATT: now also F2.2, SW2.2 (B); no longer BT3.1 (+), Q1.2 (D)
- net BUZZER: now also U3.31 (IO35); no longer U3.34 (IO38)
- net GND: now also C14.2, Q3.2 (S), Q4.1 (G), R18.2, R19.2, SW5.1, SW6.1, SW7.1, SW8.1, SW9.1, U13.2 (GND), U13.3 (CTL), U13.4 (STAT), U14.11 (GND), U14.15 (GND), U14.17 (PAD), U14.2 (GAIN_SLOT), U14.3 (GND), U4.1 (GND), U5.1 (GND); no longer R13.2
- net VBUS: now also Q4.2 (D); no longer Q1.1 (G), R13.1
- net Vin: now also C14.1, Q4.3 (S)
- net at U3.18 (IO14): now also SW5.2
- net at U3.19 (IO15): now also SW6.2
- net at U3.20 (IO16): now also SW7.2
- net at U3.21 (IO17): now also SW8.2
- net at U3.22 (IO18): now also SW9.2
- net SDA: now reaches U3.25 (IO21)
- net SDA: now also U5.4 (SDA)
- net SCL: now reaches U3.26 (IO26)
- net SCL: now also U5.3 (SCL)
- net EN: now reaches U3.28 (IO33)
- net EN: now also U11.2 (EN)
- net BACKLIGHT: now reaches U3.29 (IO34)
- net BACKLIGHT: now also Q3.1 (G), R18.1
- net DIN: now reaches U3.32 (IO36)
- net DIN: now also U14.1 (DIN)
- net BCLK: now reaches U3.33 (IO37)
- net BCLK: now also U14.16 (BCLK)
- new net: R19.1, U13.6 (SENSE)
- new net: Q1.2 (D), SW2.3 (C), U13.1 (VIN)
- new net: Q1.1 (G), U13.5 (GATE)
- new net: BT3.1 (+), F2.1
- new net: LS2.1, U14.9 (OUTP)
- new net: LS2.2, U14.10 (OUTN)
- new net: Q3.3 (D), R14.1
- new net: R14.2, U4.10 (LEDK)
- new net: R13.2, U14.4 (~{SD_MODE})
- new net LRCLK: U14.14 (LRCLK), U3.34 (IO38)
- no-connect marks 2 -> 12
Other:
- note added: "Screen"
- note added: "Speaker"
- note removed: "Buzzer"
- moved on the sheet: BT3, C16, C17, C18, D1, Q1, R17, R9, SW3, SW4, U1, U3

Commit message: Finished first rough draft
Parts:
- removed BT1, BT2: 18650, symbol Device:Battery_Cell
- removed C1, C2: 220n, symbol Device:C_Small
- removed D10: 1N4148WS, Diode_SMD:D_SOD-323_HandSoldering, symbol Diode:1N4148WS
- removed FPC1: 5034801000, easyeda2kicad:FPC-SMD_5034801000, symbol easyeda2kicad:5034801000
- removed LS1: Buzzer, easyeda2kicad:BUZ-SMD_4P-L8.5-W8.5-P8.50-BR, symbol Device:Speaker
- removed Q2, Q3: AO3400A, Package_TO_SOT_SMD:SOT-23_Handsoldering, symbol Device:Q_NMOS_GSD
- removed R1, R2, R3, R4: 10, symbol Device:R_Small
- removed R14: 1k, Resistor_SMD:R_0402_1005Metric_Pad0.72x0.64mm_HandSolder, symbol Device:R
- removed R15: 10k, Resistor_SMD:R_0805_2012Metric_Pad1.20x1.40mm_HandSolder, symbol Device:R
- removed R16: 10, Resistor_SMD:R_0603_1608Metric_Pad0.98x0.95mm_HandSolder, symbol Device:R_Small
- removed R18: 10k, Resistor_SMD:R_0402_1005Metric_Pad0.72x0.64mm_HandSolder, symbol Device:R
- removed U12: XB8089D0, easyeda2kicad:SOIC-8_L4.9-W3.9-P1.27-LS6.0-BL-EP3.3-1, symbol easyeda2kicad:XB8089D0
- removed U15: KLJ-01304T-08R07W, easyeda2kicad:BUZ-SMD_4P-L13.0-W13.0-P11.4-BL, symbol easyeda2kicad:KLJ-01304T-08R07W
- removed U2: HS17QS178RX, easyeda2kicad:OLED-SMD_10P-P0.50_HS17QS178RX, symbol easyeda2kicad:HS17QS178RX
- removed U4: HS17QS178RX, easyeda2kicad:FPC-SMD_5034801000, symbol easyeda2kicad:HS17QS178RX
- removed U6: BQ76905RGRR, easyeda2kicad:VQFN-20_L3.5-W3.5-P0.50-TL-EP2.1, symbol easyeda2kicad:BQ76905RGRR
- removed U7, U8: SIRA60DP-T1-GE3, sussymosfet:MOSFET_7DP-T1-GE3_VIS, symbol sussymosfet:SIRA60DP-T1-GE3
- C18: LCSC Part C52923 -> C14445
- R5, R8: LCSC Part C106235 -> C11702
- U14: LCSC Part (none) -> C910544
Connections:
- net +3V3: no longer R13.1
- net +5V: now also R13.1
- net GND: no longer Q4.1 (G), R19.2, U13.4 (STAT)
- net BACKLIGHT: no longer names the net of U3.29 (IO34)
- net BUZZER: no longer names the net of U3.31 (IO35)
- net DIO1: no longer names the net of U1.13 (DIO1)
- net DIO1: no longer U3.8 (IO4)
- net DIO2: no longer names the net of U1.8 (DIO2)
- net DIO2: no longer U3.11 (IO7)
- new net: Q4.1 (G), R19.2, U13.4 (STAT)
- no-connect marks 12 -> 21

Commit message: almost done :siren-thumbsup:
Parts:
- removed R17: 10k, Resistor_SMD:R_0402_1005Metric_Pad0.72x0.64mm_HandSolder, symbol Device:R
- added BT2: li-ion, easyeda2kicad:BATTERY-SMD_18650-1S-L77.1-W20.7-1, symbol Device:Battery_Cell
- added D3, D4, D5, D6, D7: D_TVS, Diode_SMD:D_SOD-923, symbol Device:D_TVS
- added R10, R11, R12, R13, R14, R2, R4, R9: 10k, Resistor_SMD:R_0402_1005Metric_Pad0.72x0.64mm_HandSolder, symbol Device:R_Small
- added U6: INA3221, Package_DFN_QFN:Texas_RGV0016A_VQFN-16-1EP_4x4mm_P0.65mm_EP2.1x2.1mm, symbol Power_Management:INA3221
- renumbered BT3 to BT1, C8 to C1, C13 to C10, C17 to C11, C18 to C12, C16 to C13, C7 to C2, C5 to C3, C10 to C4, C4 to C5, C11 to C6, C14 to C7, C3 to C8, C6 to C9, D4 to D1, D20 to D10, D21 to D11, D3 to D2, D1 to D8, D15 to D9, F2 to F1, F1 to F2, LS2 to LS1, Q4 to Q1, Q1 to Q2, R8 to R1, R13 to R15, R9 to R16, R6 to R17, R7 to R18, R5 to R3, R11 to R5, R12 to R6, R10 to R7, R19 to R8, SW2 to SW1, SW5 to SW2, SW6 to SW3, SW7 to SW4, SW8 to SW5, SW9 to SW6, SW3 to SW7, SW4 to SW8, U11 to U1, U13 to U2, U9 to U3, U5 to U4, U10 to U5, U1 to U7, U3 to U8, U14 to U9
Connections:
- net +3V3: now also D4.2 (A2), R10.1, R11.1, R12.1, R13.1, R14.1, R2.1, R4.1, R9.1, U6.16 (VPU), U6.4 (VS)
- net +5V: now also D6.2 (A2)
- net +BATT: now also D3.2 (A2), U6.12 (IN+1)
- net GND: now also BT2.2 (-), D3.1 (A1), D4.1 (A1), D5.1 (A1), D6.1 (A1), D7.1 (A1), U6.11 (IN-1), U6.17 (EP), U6.3 (GND)
- net SCL: now also D7.2 (A2), R2.2, U6.6 (SCL)
- net SDA: now also D5.2 (A2), R4.2, U6.7 (SDA)
- net Vin: now also R8.1, U2.6 (SENSE)
- net at SW2.2, U8.18 (IO14): now also R9.2
- net at SW4.2, U8.20 (IO16): now also R11.2
- net at BT1.1 (+), F1.1: now also BT2.1 (+)
- net at C12.1, SW7.2, U8.45 (EN): now also R14.2
- net at SW6.2, U8.22 (IO18): now also R13.2
- net at SW3.2, U8.19 (IO15): now also R10.2
- net at SW5.2, U8.21 (IO17): now also R12.2
- no-connect marks 21 -> 30
Other:
- moved on the sheet: C11, C12, C13, C3, C7, C9, SW2, SW3, SW4, SW5, SW6, SW7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

Commit message: Final product: version 1 has been ordered
Parts:
- added J3: Conn_01x05_Socket, Connector_PinHeader_2.54mm:PinHeader_1x05_P2.54mm_Vertical, symbol Connector:Conn_01x05_Socket
- L1: footprint Inductor_SMD_Wurth:L_Wurth_WE-LQSH-4020 -> 74438356010:WE-MAPI_4020
- U6: LCSC Part (none) -> C181255
Connections:
- net GND: now also U3.1 (TEMP)
- net SCL: now also U8.31 (IO35); no longer U8.26 (IO26)
- net SDA: now also U8.29 (IO34); no longer U8.25 (IO21)
- net IO47: now reaches U8.27 (IO47)
- net IO47: now also J3.4 (Pin_4)
- net IO48: now reaches U8.30 (IO48)
- net IO48: now also J3.5 (Pin_5)
- net IO40: now reaches U8.36 (IO40)
- net IO40: now also J3.3 (Pin_3)
- net IO41: now reaches U8.37 (IO41)
- net IO41: now also J3.2 (Pin_2)
- net IO42: now reaches U8.38 (IO42)
- net IO42: now also J3.1 (Pin_1)
- no-connect marks 30 -> 26
Other:
- note added: "These two batteries are not intended to be connected at the same time!"
- moved on the sheet: BT1, BT2, C12, C13, C3, C9, D10, D11, D3, D4, D5, D6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
